File: Split V2/Split V2/Split V2.kicad_pcb (KiCad board)
At the start: 2 copper layers, 190.5 x 153.2 mm, 61 parts

Commit message: Connected schematic and pcb
Got the Schematic and pcb linked and started searching for symbols for arduio promicro
Parts:
- added U1: ProMicro, Keebio-Parts.pretty-master:ArduinoProMicro, F.Cu at (221.0, 87.6)
- DX0,Y0: renamed from D9; value (none) -> ~
- DX0,Y1: renamed from D14; value (none) -> ~
- DX0,Y2: renamed from D19; value (none) -> ~
- DX0,Y3: renamed from D28; value (none) -> ~
- DX0,Y4: renamed from D29; value (none) -> ~
- DX0,Y5: renamed from D30; value (none) -> ~
- DX1,Y0: renamed from D1; value (none) -> ~
- DX1,Y1: renamed from D5; value (none) -> ~
- DX1,Y2: renamed from D10; value (none) -> ~
- DX1,Y3: renamed from D15; value (none) -> ~
- DX1,Y4: renamed from D20; value (none) -> ~
- DX1,Y5: renamed from D24; value (none) -> ~
- DX2,Y0: renamed from D2; value (none) -> ~
- DX2,Y1: renamed from D6; value (none) -> ~
- DX2,Y2: renamed from D11; value (none) -> ~
- DX2,Y3: renamed from D16; value (none) -> ~
- DX2,Y4: renamed from D21; value (none) -> ~
- DX2,Y5: renamed from D25; value (none) -> ~
- DX3,Y0, DX3,Y1, DX3,Y2, DX3,Y3, DX3,Y4, DX3,Y5, DX4,Y0, DX4,Y1, DX4,Y2, DX4,Y3, DX4,Y4, DX4,Y5, SWX0,Y0, SWX0,Y1, SWX0,Y2, SWX0,Y3, SWX0,Y4, SWX0,Y5, SWX1,Y0, SWX1,Y1, SWX1,Y2, SWX1,Y3, SWX2,Y0, SWX2,Y1, SWX2,Y2, SWX2,Y3, SWX2,Y4, SWX2,Y5, SWX3,Y0, SWX3,Y1, SWX3,Y2, SWX3,Y3, SWX3,Y4, SWX3,Y5, SWX4,Y0, SWX4,Y1, SWX4,Y2, SWX4,Y3, SWX4,Y5: value (none) -> ~
- SWX1,Y4: renamed from SWX1,Y3; value (none) -> ~
- SWX1,Y5: renamed from SWX1,Y4; value (none) -> ~
- SWX4,Y4: renamed from SWX4,Y5; value (none) -> ~
Connections:
- DX0,Y0 pad 1: (no net) -> unconnected-(DX0,Y0-K-Pad1)
- DX0,Y0 pad 2: (no net) -> Net-(DX0,Y0-A)
- DX0,Y1 pad 1: (no net) -> unconnected-(DX0,Y1-K-Pad1)
- DX0,Y1 pad 2: (no net) -> Net-(DX0,Y1-A)
- DX0,Y2 pad 1: (no net) -> unconnected-(DX0,Y2-K-Pad1)
- DX0,Y2 pad 2: (no net) -> Net-(DX0,Y2-A)
- DX0,Y3 pad 1: (no net) -> unconnected-(DX0,Y3-K-Pad1)
- DX0,Y3 pad 2: (no net) -> Net-(DX0,Y3-A)
- DX0,Y4 pad 1: (no net) -> unconnected-(DX0,Y4-K-Pad1)
- DX0,Y4 pad 2: (no net) -> Net-(DX0,Y4-A)
- DX0,Y5 pad 1: (no net) -> unconnected-(DX0,Y5-K-Pad1)
- DX0,Y5 pad 2: (no net) -> Net-(DX0,Y5-A)
- DX1,Y0 pad 1: (no net) -> unconnected-(DX1,Y0-K-Pad1)
- DX1,Y0 pad 2: (no net) -> Net-(DX1,Y0-A)
- DX1,Y1 pad 1: (no net) -> unconnected-(DX1,Y1-K-Pad1)
- DX1,Y1 pad 2: (no net) -> Net-(DX1,Y1-A)
- DX1,Y2 pad 1: (no net) -> unconnected-(DX1,Y2-K-Pad1)
- DX1,Y2 pad 2: (no net) -> Net-(DX1,Y2-A)
- DX1,Y3 pad 1: (no net) -> unconnected-(DX1,Y3-K-Pad1)
- DX1,Y3 pad 2: (no net) -> Net-(DX1,Y3-A)
- DX1,Y4 pad 1: (no net) -> unconnected-(DX1,Y4-K-Pad1)
- DX1,Y4 pad 2: (no net) -> Net-(DX1,Y4-A)
- DX1,Y5 pad 1: (no net) -> unconnected-(DX1,Y5-K-Pad1)
- DX1,Y5 pad 2: (no net) -> Net-(DX1,Y5-A)
- DX2,Y0 pad 1: (no net) -> unconnected-(DX2,Y0-K-Pad1)
- DX2,Y0 pad 2: (no net) -> Net-(DX2,Y0-A)
- DX2,Y1 pad 1: (no net) -> unconnected-(DX2,Y1-K-Pad1)
- DX2,Y1 pad 2: (no net) -> Net-(DX2,Y1-A)
- DX2,Y2 pad 1: (no net) -> unconnected-(DX2,Y2-K-Pad1)
- DX2,Y2 pad 2: (no net) -> Net-(DX2,Y2-A)
- DX2,Y3 pad 1: (no net) -> unconnected-(DX2,Y3-K-Pad1)
- DX2,Y3 pad 2: (no net) -> Net-(DX2,Y3-A)
- DX2,Y4 pad 1: (no net) -> unconnected-(DX2,Y4-K-Pad1)
- DX2,Y4 pad 2: (no net) -> Net-(DX2,Y4-A)
- DX2,Y5 pad 1: (no net) -> unconnected-(DX2,Y5-K-Pad1)
- DX2,Y5 pad 2: (no net) -> Net-(DX2,Y5-A)
- DX3,Y0 pad 1: (no net) -> unconnected-(DX3,Y0-K-Pad1)
- DX3,Y0 pad 2: (no net) -> Net-(DX3,Y0-A)
- DX3,Y1 pad 1: (no net) -> unconnected-(DX3,Y1-K-Pad1)
- DX3,Y1 pad 2: (no net) -> Net-(DX3,Y1-A)
- DX3,Y2 pad 1: (no net) -> unconnected-(DX3,Y2-K-Pad1)
- DX3,Y2 pad 2: (no net) -> Net-(DX3,Y2-A)
- DX3,Y3 pad 1: (no net) -> unconnected-(DX3,Y3-K-Pad1)
- DX3,Y3 pad 2: (no net) -> Net-(DX3,Y3-A)
- DX3,Y4 pad 1: (no net) -> unconnected-(DX3,Y4-K-Pad1)
- DX3,Y4 pad 2: (no net) -> Net-(DX3,Y4-A)
- DX3,Y5 pad 1: (no net) -> unconnected-(DX3,Y5-K-Pad1)
- DX3,Y5 pad 2: (no net) -> Net-(DX3,Y5-A)
- DX4,Y0 pad 1: (no net) -> unconnected-(DX4,Y0-K-Pad1)
- DX4,Y0 pad 2: (no net) -> Net-(DX4,Y0-A)
- DX4,Y1 pad 1: (no net) -> unconnected-(DX4,Y1-K-Pad1)
- DX4,Y1 pad 2: (no net) -> Net-(DX4,Y1-A)
- DX4,Y2 pad 1: (no net) -> unconnected-(DX4,Y2-K-Pad1)
- DX4,Y2 pad 2: (no net) -> Net-(DX4,Y2-A)
- DX4,Y3 pad 1: (no net) -> unconnected-(DX4,Y3-K-Pad1)
- DX4,Y3 pad 2: (no net) -> Net-(DX4,Y3-A)
- DX4,Y4 pad 1: (no net) -> unconnected-(DX4,Y4-K-Pad1)
- DX4,Y4 pad 2: (no net) -> Net-(DX4,Y4-A)
- DX4,Y5 pad 1: (no net) -> unconnected-(DX4,Y5-K-Pad1)
- DX4,Y5 pad 2: (no net) -> Net-(DX4,Y5-A)
- SWX0,Y0 pad 1: (no net) -> unconnected-(SWX0,Y0-Pad1)
- SWX0,Y0 pad 2: (no net) -> Net-(DX0,Y0-A)
- SWX0,Y1 pad 1: (no net) -> unconnected-(SWX0,Y1-Pad1)
- SWX0,Y1 pad 2: (no net) -> Net-(DX0,Y1-A)
- SWX0,Y2 pad 1: (no net) -> unconnected-(SWX0,Y2-Pad1)
- SWX0,Y2 pad 2: (no net) -> Net-(DX0,Y2-A)
- SWX0,Y3 pad 1: (no net) -> unconnected-(SWX0,Y3-Pad1)
- SWX0,Y3 pad 2: (no net) -> Net-(DX0,Y3-A)
- SWX0,Y4 pad 1: (no net) -> unconnected-(SWX0,Y4-Pad1)
- SWX0,Y4 pad 2: (no net) -> Net-(DX0,Y4-A)
- SWX0,Y5 pad 1: (no net) -> unconnected-(SWX0,Y5-Pad1)
- SWX0,Y5 pad 2: (no net) -> Net-(DX0,Y5-A)
- SWX1,Y0 pad 1: (no net) -> unconnected-(SWX1,Y0-Pad1)
- SWX1,Y0 pad 2: (no net) -> Net-(DX1,Y0-A)
- SWX1,Y1 pad 1: (no net) -> unconnected-(SWX1,Y1-Pad1)
- SWX1,Y1 pad 2: (no net) -> Net-(DX1,Y1-A)
- SWX1,Y2 pad 1: (no net) -> unconnected-(SWX1,Y2-Pad1)
- SWX1,Y2 pad 2: (no net) -> Net-(DX1,Y2-A)
- SWX1,Y3 pad 1: (no net) -> unconnected-(SWX1,Y3-Pad1)
- SWX1,Y3 pad 2: (no net) -> Net-(DX1,Y3-A)
- SWX1,Y4 pad 1: (no net) -> unconnected-(SWX1,Y4-Pad1)
- SWX1,Y4 pad 2: (no net) -> Net-(DX1,Y4-A)
- SWX1,Y5 pad 1: (no net) -> unconnected-(SWX1,Y5-Pad1)
- SWX1,Y5 pad 2: (no net) -> Net-(DX1,Y5-A)
- SWX2,Y0 pad 1: (no net) -> unconnected-(SWX2,Y0-Pad1)
- SWX2,Y0 pad 2: (no net) -> Net-(DX2,Y0-A)
- SWX2,Y1 pad 1: (no net) -> unconnected-(SWX2,Y1-Pad1)
- SWX2,Y1 pad 2: (no net) -> Net-(DX2,Y1-A)
- SWX2,Y2 pad 1: (no net) -> unconnected-(SWX2,Y2-Pad1)
- SWX2,Y2 pad 2: (no net) -> Net-(DX2,Y2-A)
- SWX2,Y3 pad 1: (no net) -> unconnected-(SWX2,Y3-Pad1)
- SWX2,Y3 pad 2: (no net) -> Net-(DX2,Y3-A)
- SWX2,Y4 pad 1: (no net) -> unconnected-(SWX2,Y4-Pad1)
- SWX2,Y4 pad 2: (no net) -> Net-(DX2,Y4-A)
- SWX2,Y5 pad 1: (no net) -> unconnected-(SWX2,Y5-Pad1)
- SWX2,Y5 pad 2: (no net) -> Net-(DX2,Y5-A)
- SWX3,Y0 pad 1: (no net) -> unconnected-(SWX3,Y0-Pad1)
- SWX3,Y0 pad 2: (no net) -> Net-(DX3,Y0-A)
- SWX3,Y1 pad 1: (no net) -> unconnected-(SWX3,Y1-Pad1)
- SWX3,Y1 pad 2: (no net) -> Net-(DX3,Y1-A)
- SWX3,Y2 pad 1: (no net) -> unconnected-(SWX3,Y2-Pad1)
- SWX3,Y2 pad 2: (no net) -> Net-(DX3,Y2-A)
- SWX3,Y3 pad 1: (no net) -> unconnected-(SWX3,Y3-Pad1)
- SWX3,Y3 pad 2: (no net) -> Net-(DX3,Y3-A)
- SWX3,Y4 pad 1: (no net) -> unconnected-(SWX3,Y4-Pad1)
- SWX3,Y4 pad 2: (no net) -> Net-(DX3,Y4-A)
- SWX3,Y5 pad 1: (no net) -> unconnected-(SWX3,Y5-Pad1)
- SWX3,Y5 pad 2: (no net) -> Net-(DX3,Y5-A)
- SWX4,Y0 pad 1: (no net) -> unconnected-(SWX4,Y0-Pad1)
- SWX4,Y0 pad 2: (no net) -> Net-(DX4,Y0-A)
- SWX4,Y1 pad 1: (no net) -> unconnected-(SWX4,Y1-Pad1)
- SWX4,Y1 pad 2: (no net) -> Net-(DX4,Y1-A)
- SWX4,Y2 pad 1: (no net) -> unconnected-(SWX4,Y2-Pad1)
- SWX4,Y2 pad 2: (no net) -> Net-(DX4,Y2-A)
- SWX4,Y3 pad 1: (no net) -> unconnected-(SWX4,Y3-Pad1)
- SWX4,Y3 pad 2: (no net) -> Net-(DX4,Y3-A)
- SWX4,Y4 pad 1: (no net) -> unconnected-(SWX4,Y4-Pad1)
- SWX4,Y4 pad 2: (no net) -> Net-(DX4,Y4-A)
- SWX4,Y5 pad 1: (no net) -> unconnected-(SWX4,Y5-Pad1)
- SWX4,Y5 pad 2: (no net) -> Net-(DX4,Y5-A)
