File: Archive/kicad/board/board.kicad_pcb (KiCad board)
At the start: 2 copper layers, 126.9 x 103.7 mm, 39 parts

Commit message: V1 Traces
Got all of my traces layed out and worked on creating the reversable footprint like in other projects. Need to do some more research as to the specifics
Parts:
- moved D1 200.6 mm to (166.3, 126.1)
- moved D10 200.6 mm to (221.3, 121.9)
- moved D11 200.6 mm to (222.9, 104.0)
- moved D12 200.6 mm to (224.5, 86.1)
- moved D13 200.6 mm to (239.1, 125.5)
- moved D14 200.6 mm to (240.6, 107.6)
- moved D15 200.6 mm to (242.2, 89.6)
- moved D16 200.6 mm to (230.4, 143.8)
- moved D17 200.6 mm to (248.8, 149.6)
- moved D18 200.6 mm to (265.1, 159.8)
- moved D2 200.6 mm to (166.3, 108.1)
- moved D3 200.6 mm to (166.3, 90.1)
- moved D4 200.6 mm to (185.5, 117.8)
- moved D5 200.6 mm to (187.1, 99.9)
- moved D6 200.6 mm to (188.7, 81.9)
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