File: Split Cherry/Split Cherry.kicad_sch (KiCad schematic)
At the start: 67 parts, among them J1 AudioJack4

Commit message: Modified Split and made new
Modified the original split to correct ADC error for joystick and started work on a Split keyboard with cherry switches
Parts:
- SWML1, SWMR1, SWX0,Y0, SWX0,Y1, SWX0,Y2, SWX0,Y3, SWX0,Y4, SWX0,Y5, SWX1,Y0, SWX1,Y1, SWX1,Y2, SWX1,Y3, SWX1,Y4, SWX1,Y5, SWX2,Y0, SWX2,Y1, SWX2,Y2, SWX2,Y3, SWX2,Y4, SWX2,Y5, SWX3,Y0, SWX3,Y1, SWX3,Y2, SWX3,Y3, SWX3,Y4, SWX3,Y5, SWX4,Y0, SWX4,Y1, SWX4,Y2, SWX4,Y3, SWX4,Y4, SWX4,Y5: footprint keyswitches.pretty-master:Kailh_socket_PG1350_optional_reversible -> Keys pretty:SW_MX_reversible
Changed lines of the file:
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@@
 			)
 		)
-		(property "Footprint" "keyswitches.pretty-master:Kailh_socket_PG1350_optional_reversible"
+		(property "Footprint" "Keys pretty:SW_MX_reversible"
 			(at 88.9 52.07 0)
 			(effects
@@
 			)
 		)
-		(property "Footprint" "keyswitches.pretty-master:Kailh_socket_PG1350_optional_reversible"
+		(property "Footprint" "Keys pretty:SW_MX_reversible"
 			(at 139.7 64.77 0)
 			(effects
@@
 			)
 		)
-		(property "Footprint" "keyswitches.pretty-master:Kailh_socket_PG1350_optional_reversible"
+		(property "Footprint" "Keys pretty:SW_MX_reversible"
 			(at 71.12 52.07 0)
 			(effects
@@
 			)
 		)
-		(property "Footprint" "keyswitches.pretty-master:Kailh_socket_PG1350_optional_reversible"
+		(property "Footprint" "Keys pretty:SW_MX_reversible"
 			(at 139.7 77.47 0)
 			(effects
@@
 			)
 		)
-		(property "Footprint" "keyswitches.pretty-master:Kailh_socket_PG1350_optional_reversible"
+		(property "Footprint" "Keys pretty:SW_MX_reversible"
 			(at 123.19 77.47 0)
 			(effects
@@
 			)
 		)
-		(property "Footprint" "keyswitches.pretty-master:Kailh_socket_PG1350_optional_reversible"
+		(property "Footprint" "Keys pretty:SW_MX_reversible"
 			(at 105.41 102.87 0)
 			(effects
@@
 			)
 		)
-		(property "Footprint" "keyswitches.pretty-master:Kailh_socket_PG1350_optional_reversible"
+		(property "Footprint" "Keys pretty:SW_MX_reversible"
 			(at 123.19 102.87 0)
 			(effects
@@
 			)
 		)
-		(property "Footprint" "keyswitches.pretty-master:Kailh_socket_PG1350_optional_reversible"
+		(property "Footprint" "Keys pretty:SW_MX_reversible"
 			(at 123.19 52.07 0)
 			(effects
@@
 			)
 		)
-		(property "Footprint" "keyswitches.pretty-master:Kailh_socket_PG1350_optional_reversible"
+		(property "Footprint" "Keys pretty:SW_MX_reversible"
 			(at 105.41 77.47 0)
 			(effects
@@
 			)
 		)
-		(property "Footprint" "keyswitches.pretty-master:Kailh_socket_PG1350_optional_reversible"
+		(property "Footprint" "Keys pretty:SW_MX_reversible"
 			(at 105.41 64.77 0)
 			(effects
@@
 			)
 		)
-		(property "Footprint" "keyswitches.pretty-master:Kailh_socket_PG1350_optional_reversible"
+		(property "Footprint" "Keys pretty:SW_MX_reversible"
 			(at 105.41 90.17 0)
 			(effects
@@
 			)
 		)
-		(property "Footprint" "keyswitches.pretty-master:Kailh_socket_PG1350_optional_reversible"
+		(property "Footprint" "Keys pretty:SW_MX_reversible"
 			(at 123.19 64.77 0)
 			(effects
@@
 			)
 		)
-		(property "Footprint" "keyswitches.pretty-master:Kailh_socket_PG1350_optional_reversible"
+		(property "Footprint" "Keys pretty:SW_MX_reversible"
 			(at 49.53 52.07 0)
 			(effects
@@
 			)
 		)
-		(property "Footprint" "keyswitches.pretty-master:Kailh_socket_PG1350_optional_reversible"
+		(property "Footprint" "Keys pretty:SW_MX_reversible"
 			(at 176.53 90.17 0)
 			(effects
@@
 			)
 		)
-		(property "Footprint" "keyswitches.pretty-master:Kailh_socket_PG1350_optional_reversible"
+		(property "Footprint" "Keys pretty:SW_MX_reversible"
 			(at 71.12 102.87 0)
 			(effects
@@
 			)
 		)
-		(property "Footprint" "keyswitches.pretty-master:Kailh_socket_PG1350_optional_reversible"
+		(property "Footprint" "Keys pretty:SW_MX_reversible"
 			(at 139.7 102.87 0)
 			(effects
@@
 			)
 		)
-		(property "Footprint" "keyswitches.pretty-master:Kailh_socket_PG1350_optional_reversible"
+		(property "Footprint" "Keys pretty:SW_MX_reversible"
 			(at 105.41 52.07 0)
 			(effects
@@
 			)
 		)
-		(property "Footprint" "keyswitches.pretty-master:Kailh_socket_PG1350_optional_reversible"
+		(property "Footprint" "Keys pretty:SW_MX_reversible"
 			(at 139.7 90.17 0)
 			(effects
@@
 			)
 		)
-		(property "Footprint" "keyswitches.pretty-master:Kailh_socket_PG1350_optional_reversible"
+		(property "Footprint" "Keys pretty:SW_MX_reversible"
 			(at 49.53 64.77 0)
 			(effects
@@
 			)
 		)
-		(property "Footprint" "keyswitches.pretty-master:Kailh_socket_PG1350_optional_reversible"
+		(property "Footprint" "Keys pretty:SW_MX_reversible"
 			(at 193.04 90.17 0)
 			(effects
@@
 			)
 		)
-		(property "Footprint" "keyswitches.pretty-master:Kailh_socket_PG1350_optional_reversible"
+		(property "Footprint" "Keys pretty:SW_MX_reversible"
 			(at 88.9 64.77 0)
 			(effects
@@
 			)
 		)
-		(property "Footprint" "keyswitches.pretty-master:Kailh_socket_PG1350_optional_reversible"
+		(property "Footprint" "Keys pretty:SW_MX_reversible"
 			(at 139.7 52.07 0)
 			(effects
@@
 			)
 		)
-		(property "Footprint" "keyswitches.pretty-master:Kailh_socket_PG1350_optional_reversible"
+		(property "Footprint" "Keys pretty:SW_MX_reversible"
 			(at 88.9 77.47 0)
 			(effects
@@
 			)
 		)
-		(property "Footprint" "keyswitches.pretty-master:Kailh_socket_PG1350_optional_reversible"
+		(property "Footprint" "Keys pretty:SW_MX_reversible"
 			(at 88.9 90.17 0)
 			(effects
@@
 			)
 		)
-		(property "Footprint" "keyswitches.pretty-master:Kailh_socket_PG1350_optional_reversible"
+		(property "Footprint" "Keys pretty:SW_MX_reversible"
 			(at 49.53 102.87 0)
 			(effects
@@
 			)
 		)
-		(property "Footprint" "keyswitches.pretty-master:Kailh_socket_PG1350_optional_reversible"
+		(property "Footprint" "Keys pretty:SW_MX_reversible"
 			(at 71.12 64.77 0)
 			(effects
@@
 			)
 		)
-		(property "Footprint" "keyswitches.pretty-master:Kailh_socket_PG1350_optional_reversible"
+		(property "Footprint" "Keys pretty:SW_MX_reversible"
 			(at 123.19 90.17 0)
 			(effects
@@
 			)
 		)
-		(property "Footprint" "keyswitches.pretty-master:Kailh_socket_PG1350_optional_reversible"
+		(property "Footprint" "Keys pretty:SW_MX_reversible"
 			(at 71.12 77.47 0)
 			(effects
@@
 			)
 		)
-		(property "Footprint" "keyswitches.pretty-master:Kailh_socket_PG1350_optional_reversible"
+		(property "Footprint" "Keys pretty:SW_MX_reversible"
 			(at 49.53 90.17 0)
 			(effects
@@
 			)
 		)
-		(property "Footprint" "keyswitches.pretty-master:Kailh_socket_PG1350_optional_reversible"
+		(property "Footprint" "Keys pretty:SW_MX_reversible"
 			(at 88.9 102.87 0)
 			(effects
@@
 			)
 		)
-		(property "Footprint" "keyswitches.pretty-master:Kailh_socket_PG1350_optional_reversible"
+		(property "Footprint" "Keys pretty:SW_MX_reversible"
 			(at 49.53 77.47 0)
 			(effects
@@
 			)
 		)
-		(property "Footprint" "keyswitches.pretty-master:Kailh_socket_PG1350_optional_reversible"
+		(property "Footprint" "Keys pretty:SW_MX_reversible"
 			(at 71.12 90.17 0)
 			(effects
